Commit message: add marker

File: husky_description/urdf/husky.urdf.xacro (robot description, xacro)
@@ -40,4 +40,5 @@
   <xacro:include filename="$(find husky_description)/urdf/accessories/sick_lms1xx_mount.urdf.xacro"/>
   <xacro:include filename="$(find husky_description)/urdf/accessories/sensor_arch.urdf.xacro"/>
+  <xacro:include filename="$(find husky_description)/urdf/accessories/marker_mount.urdf.xacro"/>
   <xacro:property name="M_PI" value="3.14159"/>
   <!-- Base Size -->
@@ -134,4 +135,10 @@
     </xacro:sensor_arch>
   </xacro:if>
+  <!--Custom-->
+  <xacro:if value="$(arg marker_enabled)">
+    <xacro:marker_mount prefix="" parent="top_plate_link">
+      <origin xyz="-0.35 0 0.25" rpy="0 0 -3.14"/>
+    </xacro:marker_mount>
+  </xacro:if>
   <!-- add the intel realsense to the topbar if needed -->
   <xacro:if value="$(arg realsense_enabled)">
