Commit message: add package

File: husky_description/urdf/accessories/intel_realsense.urdf.xacro (robot description, xacro)
@@ -80,5 +80,5 @@
           <mesh filename="package://realsense2_description/meshes/d415.stl" />
         </geometry>
-        <material name="white" />
+        <material name="yellow" />
       </visual>
     </link>
